Commit message: Adding more structure

File: urdf/board.urdf.xacro (robot description, xacro)
@@ -3,5 +3,5 @@
   <gazebo>
     <plugin name="hand_of_god" filename="libgazebo_ros_hand_of_god.so">
-      <linkName>checkerboard</linkName>
+      <linkName>board_link</linkName>
       <frameId>hog</frameId>
       <kl>200</kl>
@@ -9,5 +9,5 @@
     </plugin>
   </gazebo>
-  <link name="checkerboard">
+  <link name="board_link">
     <collision>
       <geometry>

File: urdf/camera.urdf.xacro (robot description, xacro)
@@ -29,4 +29,16 @@
     </inertial>
   </link>
+  <joint name="camera_optical_joint" type="fixed">
+    <origin xyz="0 0 0" rpy="-1.5707 0 -1.5707"/>
+    <parent link="camera_link"/>
+    <child link="camera_optical_link"/>
+  </joint>
+  <link name="camera_optical_link">
+    <inertial>
+      <mass value="1e-5" />
+      <origin xyz="0 0 0" rpy="0 0 0"/>
+      <inertia ixx="1e-6" ixy="0" ixz="0" iyy="1e-6" iyz="0" izz="1e-6" />
+    </inertial>
+  </link>
   <!-- camera -->
   <gazebo reference="camera_link">
@@ -34,4 +46,5 @@
       <update_rate>30.0</update_rate>
       <camera name="head">
+        <!-- 50-degree FOV -->
         <horizontal_fov>0.873</horizontal_fov>
         <image>
@@ -46,12 +59,9 @@
         <noise>
           <type>gaussian</type>
-          <!-- Noise is sampled independently per pixel on each frame.
-               That pixel's noise value is added to each of its color
-               channels, which at that point lie in the range [0,1]. -->
           <mean>0.0</mean>
           <stddev>0.007</stddev>
         </noise>
       </camera>
-      <plugin name="camera_controller" filename="libgazebo_ros_camera.so">
+      <plugin name="camera_sensor" filename="libgazebo_ros_camera.so">
         <alwaysOn>true</alwaysOn>
         <updateRate>0.0</updateRate>
@@ -59,5 +69,5 @@
         <imageTopicName>image_raw</imageTopicName>
         <cameraInfoTopicName>camera_info</cameraInfoTopicName>
-        <frameName>camera_link</frameName>
+        <frameName>camera_optical_link</frameName>
         <hackBaseline>0.07</hackBaseline>
         <distortionK1>0.0</distortionK1>
